Commit message: fix target range, add plane positioning, cube size

File: pybullet_multigoal_gym/assets/robots/kuka/iiwa14_parallel_jaw_cube.urdf (robot description, URDF)
Before this commit: robot iiwa14, 18 links, 17 joints
Links:
- link base_cube: geometry collision box size=0.5 0.5 0.5; visual box size=0.5 0.5 0.5
Joints:
- joint cube_iiwa_joint: origin xyz=0 0 -0.5 rpy=0 0 0 -> xyz=0 0 -0.25 rpy=0 0 0
