Commit message: add spring usecase

File: pybullet_multigoal_gym/assets/objects/assembling_shape/sphere.urdf (robot description, URDF)
Before this commit: robot cube, 1 links, 0 joints
Links:
- removed link baseLink
- added link base_link, mass .1; collision sphere radius=0.5; visual mesh filename=textured_sphere_smooth.obj scale=0.5 0.5 0.5

File: pybullet_multigoal_gym/assets/robots/kuka/iiwa14_parallel_jaw_cube.urdf (robot description, URDF)
Before this commit: robot iiwa14, 18 links, 17 joints
Links:
- link base_cube: mass 1.0 -> 10.0

Commit message: fix spring env

File: pybullet_multigoal_gym/assets/objects/assembling_shape/sphere.urdf (robot description, URDF)
Before this commit: robot urdf_robot, 1 links, 0 joints
Links:
- link base_link: geometry collision sphere radius=1.0; visual mesh filename=textured_sphere_smooth.obj scale=1.0 1.0 1.0
